File: kicad-c16-multirom/kicad-c16-multirom.kicad_sch (KiCad schematic)
At the start: 12 parts, among them J1 Conn_01x02_Pin, J2 Conn_01x02_Pin, J3 Conn_01x01_Pin, J4 Conn_01x01_Pin, J5 Conn_01x01_Pin, U1 ATtiny85-20P, U2 74LS00, U3 27C512, U4 27C512

Commit message: ATTiny code updated and tested, clarified on schematics how to connect /RESET line
Other:
- note added: "~{RESET} from U15 pin 1 or U9 pin 2 or vias near U14 pin 11"
- note removed: "~{RESET} from U15 pin 1 or vias near U14 pin 11 or U9 pin 2"
Changed lines of the file:
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@@
 		)
 	)
-	(text "~{RESET} from U15 pin 1\nor vias near U14 pin 11\nor U9 pin 2"
+	(text "~{RESET} from U15 pin 1\nor U9 pin 2\nor vias near U14 pin 11\n"
 		(exclude_from_sim no)
 		(at 253.746 132.842 0)
